Commit message: frontier_exploration added

File: src/aura_description/urdf/sensors.xacro (robot description, xacro)
@@ -5,5 +5,5 @@
     base_link is the IMU-center reference frame.
     imu_link:   (0, 0, 0)     relative to base_link
-    laser_link: (0, 0, 0.178) relative to base_link
+    laser_frame: (0, 0, 0.178) relative to base_link
   -->
   <!-- IMU sensor — coincident with base_link -->
@@ -15,5 +15,5 @@
   </joint>
   <!-- LiDAR sensor — mounted on top of the robot -->
-  <link name="laser_link">
+  <link name="laser_frame">
     <visual>
       <geometry>
@@ -39,5 +39,5 @@
   <joint name="laser_joint" type="fixed">
     <parent link="base_link"/>
-    <child  link="laser_link"/>
+    <child  link="laser_frame"/>
     <origin xyz="0 0 0.178" rpy="0 0 0"/>
   </joint>
